File: Electronics/PowerSupply/Schematic/PowerDriver.sch (KiCad schematic (older format))
At the start: 48 parts, among them J1 +12V, J2 GND, J3 Scope, J4 Disable, J5 XDUCER, P10 CONN_1, P11 CONN_1, P12 CONN_1, P13 CONN_1, P14 CONN_1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

Commit message: Completed Board layout and generated gerber files.
Parts:
- removed C4: 100nF, Capacitors_SMD:C_0805_HandSoldering, symbol C_Small
